File: Kicad/AD5M.kicad_pcb (KiCad board)
At the start: 2 copper layers, 50 x 55 mm, 16 parts, among them J1 Vin, J2 Conn_01x11, J3 Ext, U1 LMR14006Y, U2 ESP32 C3 SuperMini, U5 DRV8871 Module, U6 DRV8871 Module

Commit message: Fixed ESP32 footprint & symbol Updated KiCad files Updated gerbers to board version 1.1
Parts:
- D1: footprint Diode_SMD:D_SOD-123 -> Diode_SMD:D_SOD-323
Connections:
- U2 pad 10: GND -> FAN_EXHAUST
- U2 pad 11: 3.3V -> TVOC_LED
- U2 pad 12: 4 -> 3
- U2 pad 13: 3 -> 4
- U2 pad 14: TVOC_LED -> 3.3V
- U2 pad 15: FAN_EXHAUST -> GND
- U2 pad 16: FAN_RECIRC -> 5V
- U2 pad 9: 5V -> FAN_RECIRC
Routing:
- net FAN_RECIRC: track 35.8 -> 22.8 mm, vias 0 -> 1
- net FAN_EXHAUST: track 20.2 -> 11.0 mm, vias 0 -> 1
- net 5V: track 74.0 -> 83.0 mm, vias 1 -> 0
- net TVOC_LED: track 18.4 -> 10.7 mm
- net 3.3V: track 42.1 -> 47.5 mm, vias 3 -> 4
- net 3: track 21.9 -> 24.0 mm, vias 2 -> 1
- net 4: track 22.8 -> 24.7 mm, vias 2 -> 1
- net 5: track 20.2 -> 21.5 mm
- net 7: track 21.3 -> 20.2 mm, vias 1 -> 2
- net GND: track 19.0 -> 19.6 mm, vias 46 -> 63
Other:
- board text added: "V1.1"
- board text removed: "V1.0"
